Commit message: add wheels

File: my_robo.urdf (robot description, URDF)
Before this commit: robot my_robo, 1 links, 0 joints
Links:
- added link base_footprint
- added link caster_link; visual sphere radius=0.05
- added link left_wheel_link; visual cylinder length=0.05 radius=0.1
- added link right_wheel_link; visual cylinder length=0.05 radius=0.1
Joints:
- added joint base_link_joint: type fixed, parent base_footprint, child base_link, origin xyz=0 0 0.100
- added joint caster_joint: type fixed, parent base_link, child caster_link, origin xyz=0.150 0 -0.050
- added joint left_wheel_joint: type continuous, parent base_link, child left_wheel_link, origin xyz=-0.100 0.130 0 rpy=-1.5707 0 0, axis 0 0 1
- added joint right_wheel_joint: type continuous, parent base_link, child right_wheel_link, origin xyz=-0.100 -0.130 0 rpy=1.5707 0 0, axis 0 0 1

Commit message: GAZEBOで走るようになった

File: my_robo.urdf (robot description, URDF)
Before this commit: robot my_robo, 5 links, 4 joints
Links:
- link base_link: mass None -> 0.500
- link caster_link: mass None -> 0.500; geometry collision sphere radius=0.05; visual sphere radius=0.05
- link left_wheel_link: mass None -> 0.500; geometry collision cylinder length=0.05 radius=0.1; visual cylinder length=0.05 radius=0.1
- link right_wheel_link: mass None -> 0.500; geometry collision cylinder length=0.05 radius=0.1; visual cylinder length=0.05 radius=0.1
Joints:
- joint right_wheel_joint: axis 0 0 1 -> 0 0 -1

Commit message: add a camera

File: my_robo.urdf (robot description, URDF)
Before this commit: robot my_robo, 5 links, 4 joints
Links:
- added link camera_link, mass 1e-5; collision box size=0.1 0.1 0.1; visual box size=0.1 0.1 0.1
Joints:
- added joint camera_joint: type fixed, parent base_link, child camera_link, origin xyz=0 0 0.1 rpy=0 0 0, axis 0 1 0
